File: main.kicad_pcb (KiCad board)
At the start: 4 copper layers, 100 x 100 mm, 34 parts, among them J101 XT60PW-M, J102 Conn_02x10_Row_Letter_First, U203 LMR51430 500kHz, U301 INA226, U401 INA226

Commit message: fix path for external components
Parts:
- F101: footprint main.ki:FUSE_01530007Z -> PRJ:FUSE_01530007Z
- J102: footprint main.ki:PCN10C-20S-2.54DS -> PRJ:PCN10C-20S-2.54DS
- L201: footprint main.ki:WE-XHMI_6060 -> PRJ:WE-XHMI_6060
Changed lines of the file:
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@@
 		)
 		(embedded_fonts no)
-		(model "footprints/XT60PW-M.step"
+		(model "${KIPRJMOD}/3d-models/XT60PW-M.step"
 			(offset
 				(xyz 3.6 6 0)
@@
 		)
 	)
-	(footprint "main.ki:WE-XHMI_6060"
+	(footprint "PRJ:WE-XHMI_6060"
 		(layer "F.Cu")
 		(at 153.543 105.156)
@@
 		)
 	)
-	(footprint "main.ki:FUSE_01530007Z"
+	(footprint "PRJ:FUSE_01530007Z"
 		(layer "F.Cu")
 		(at 104.2329 80.518 -90)
@@
 		(embedded_fonts no)
 	)
-	(footprint "main.ki:PCN10C-20S-2.54DS"
+	(footprint "PRJ:PCN10C-20S-2.54DS"
 		(layer "F.Cu")
 		(at 193.294 79.21 -90)
@@
 		)
 		(embedded_fonts no)
-		(model "footprints//PCN10C-20S-2.54DS.stp"
+		(model "${KIPRJMOD}/3d-models/PCN10C-20S-2.54DS.stp"
 			(offset
 				(xyz -71.7 1.2 8.3)
