File: 5V.kicad_sch (KiCad schematic)
At the start: 13 parts, among them U203 LMR51430 500kHz

Commit message: fix(sch): add title_block with <<VERSION>> placeholder to all 3 schematics
PowerBoard's schematics never had a title_block at all — the version
field stayed empty in the rendered schematic PDF even after Phase 3
placeholder migration, because there was no <<VERSION>> token to
substitute.

All other 5 HW-Module-* repos follow the convention:

  (title_block
    (title "<sheet name>")
    (rev "<<VERSION>>")
    (company "Amateurfunkclub für Remote Stationen")
  )

Insert the same block into PowerBoard.kicad_sch, 5V.kicad_sch and
power_measurement.kicad_sch with sheet-appropriate titles.

Surfaced when the v1.0 deploy showed the version on the PCB silkscreen
but the schematic PDF title block remained blank.

Co-Authored-By: Claude Opus 4.7 <noreply@anthropic.com>
Other:
- company: (none) -> Amateurfunkclub für Remote Stationen
- title: (none) -> 5V Buck Converter
Changed lines of the file:
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@@
 	(generator_version "9.0")
 	(paper "A4")
+	(title_block
+		(title "5V Buck Converter")
+		(rev "<<VERSION>>")
+		(company "Amateurfunkclub für Remote Stationen")
+	)
 	(text "All CAPS should be of type X7R!"
 		(exclude_from_sim no)
