File: power_measurement.kicad_sch (KiCad schematic)
At the start: 3 parts, among them U301 INA226

Commit message: fix(sch): add title_block with <<VERSION>> placeholder to all 3 schematics
PowerBoard's schematics never had a title_block at all — the version
field stayed empty in the rendered schematic PDF even after Phase 3
placeholder migration, because there was no <<VERSION>> token to
substitute.

All other 5 HW-Module-* repos follow the convention:

  (title_block
    (title "<sheet name>")
    (rev "<<VERSION>>")
    (company "Amateurfunkclub für Remote Stationen")
  )

Insert the same block into PowerBoard.kicad_sch, 5V.kicad_sch and
power_measurement.kicad_sch with sheet-appropriate titles.

Surfaced when the v1.0 deploy showed the version on the PCB silkscreen
but the schematic PDF title block remained blank.

Co-Authored-By: Claude Opus 4.7 <noreply@anthropic.com>
Other:
- company: (none) -> Amateurfunkclub für Remote Stationen
- title: (none) -> Power Measurement
Changed lines of the file:
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@@
 	(generator_version "9.0")
 	(paper "A4")
+	(title_block
+		(title "Power Measurement")
+		(rev "<<VERSION>>")
+		(company "Amateurfunkclub für Remote Stationen")
+	)
 	(junction
 		(at 121.92 82.55)
